File: Electronics/Demo.kicad_pcb (KiCad board)
At the start: 2 copper layers, 61 x 49 mm, 27 parts, among them J1 RJ10, J2 RJ10, J3 Conn_01x02_Male, J4 PWR, SW1 SW_Push, SW2 SW_Push, SW3 SW_Push, U1 MCP2551-I-SN, U2 MCP2515-xSO, Y1 8MHz

Commit message: Duplicate work.
Parts:
- D3: footprint Diode_SMD:D_SMB-SMC_Universal_Handsoldering -> Diode_SMD:D_SMA_Handsoldering
- J3: footprint Connector_PinHeader_1.00mm:PinHeader_1x02_P1.00mm_Vertical -> Connector_PinHeader_2.54mm:PinHeader_1x02_P2.54mm_Vertical
- moved J3 1.25 mm to (144.2, 98.0)
Routing:
- net /CANL: track 26.4 -> 29.3 mm
- net Net-(J3-Pad1): track 4.76 -> 3.76 mm
- net +5V: track 138.5 -> 139.3 mm
- net /XCDR_RST: track 28.8 -> 29.5 mm
- net GND: track 207.3 -> 206.8 mm
